Commit message: Fix holonomic movement using VelocityControl and simplified physics

File: src/robot_gazebo/urdf/robot.gazebo.xacro (robot description, xacro)
@@ -11,49 +11,6 @@
     <!-- camera -->
     <xacro:include filename="$(find robot_gazebo)/urdf/camera.gazebo.xacro"/>
-    <!-- ROS2 Control -->
-    <ros2_control name="IgnitionSystem" type="system">
-      <hardware>
-        <plugin>gz_ros2_control/GazeboSimSystem</plugin>
-      </hardware>
-      <joint name="front_left_joint">
-        <command_interface name="velocity">
-          <param name="min">-10</param>
-          <param name="max">10</param>
-        </command_interface>
-        <state_interface name="position"/>
-        <state_interface name="velocity"/>
-      </joint>
-      <joint name="front_right_joint">
-        <command_interface name="velocity">
-          <param name="min">-10</param>
-          <param name="max">10</param>
-        </command_interface>
-        <state_interface name="position"/>
-        <state_interface name="velocity"/>
-      </joint>
-      <joint name="rear_left_joint">
-        <command_interface name="velocity">
-          <param name="min">-10</param>
-          <param name="max">10</param>
-        </command_interface>
-        <state_interface name="position"/>
-        <state_interface name="velocity"/>
-      </joint>
-      <joint name="rear_right_joint">
-        <command_interface name="velocity">
-          <param name="min">-10</param>
-          <param name="max">10</param>
-        </command_interface>
-        <state_interface name="position"/>
-        <state_interface name="velocity"/>
-      </joint>
-    </ros2_control>
     <gazebo>
         <!-- Joint state publisher -->
-        <plugin filename="gz_ros2_control-system"
-                name="gz_ros2_control::GazeboSimROS2ControlPlugin">
-          <parameters>$(find robot_gazebo)/config/robot_config.yaml</parameters>
-        </plugin>
-        <!-- joint -->
         <plugin filename="libignition-gazebo-joint-state-publisher-system.so" name="ignition::gazebo::systems::JointStatePublisher">
             <topic>joint_states</topic>
@@ -65,34 +22,11 @@
         <!-- imu -->
         <plugin filename="ignition-gazebo-imu-system" name="ignition::gazebo::systems::Imu"></plugin>
-        <!-- odom -->
-        <plugin
-            filename="ignition-gazebo-odometry-publisher-system"
-            name="ignition::gazebo::systems::OdometryPublisher">
-            <odom_publish_frequency>50</odom_publish_frequency>
-            <odom_topic>/odom</odom_topic>
-            <odom_frame>odom</odom_frame>
-            <robot_base_frame>base_footprint</robot_base_frame>
-            <tf_topic>/odom/tf</tf_topic>
-        </plugin>
-        <!-- Holonomic plugin -->
-        <!-- <xacro:if value="$(arg sim_ign)">
-            <plugin filename="libHolonomicPlugin.so" name="holonomic_sim::HolonomicPlugin">
-                <wheel_joint>wheel_joint</wheel_joint>
-                <top_base_joint>top_wheel_base_joint</top_base_joint>
-                <bottom_base_joint>bottom_wheel_base_joint</bottom_base_joint>
-            </plugin>
-        </xacro:if> -->
-    <plugin filename="ignition-gazebo-mecanum-drive-system" name="ignition::gazebo::systems::MecanumDrive">
-        <front_left_joint>front_left_joint</front_left_joint>
-        <front_right_joint>front_right_joint</front_right_joint>
-        <back_left_joint>rear_left_joint</back_left_joint>
-        <back_right_joint>rear_right_joint</back_right_joint>
-        <wheel_separation>0.34</wheel_separation>
-        <wheelbase>0.3</wheelbase>
-        <wheel_radius>0.05</wheel_radius>
-	<topic>/controller/cmd_vel</topic>
-        <odom_topic>/odom</odom_topic>
-        <frame_id>odom</frame_id>
-        <child_frame_id>base_link</child_frame_id>
+        <!-- Planar Move Plugin: Directly controls base velocity for holonomic movement, bypassing wheel physics -->
+        <!-- Velocity Control Plugin: Directly controls base velocity for holonomic movement -->
+        <plugin filename="libignition-gazebo-velocity-control-system.so" name="ignition::gazebo::systems::VelocityControl">
+            <topic>/controller/cmd_vel</topic>
+            <initial_linear>0 0 0</initial_linear>
+            <initial_angular>0 0 0</initial_angular>
+            <link_name>base_footprint</link_name>
         </plugin>
     </gazebo>

File: src/robot_gazebo/urdf/wheel.xacro (robot description, xacro)
@@ -6,5 +6,5 @@
   <xacro:property name="WHEEL_VISUAL_ENABLE" value="true" />
   <!-- ============================================== -->
-  <xacro:macro name="mecanum_wheel" params="name x y">
+  <xacro:macro name="mecanum_wheel" params="name x y fdir">
     <link name="${name}_link">
       <xacro:if value="${WHEEL_VISUAL_ENABLE}">
@@ -32,6 +32,7 @@
     </joint>
     <gazebo reference="${name}_link">
-      <mu1>10.0</mu1>
-      <mu2>10.0</mu2>
+      <mu1>0.001</mu1>
+      <mu2>0.001</mu2>
+      <fdir1>${fdir}</fdir1>
       <kp>1000000000.0</kp>
       <kd>100000.0</kd>
@@ -40,7 +41,10 @@
   </xacro:macro>
   <!-- ============================================== -->
-  <xacro:mecanum_wheel name="front_left"  x="0.08"  y="0.09"/>
-  <xacro:mecanum_wheel name="front_right" x="0.08"  y="-0.09"/>
-  <xacro:mecanum_wheel name="rear_left"   x="-0.08" y="0.09"/>
-  <xacro:mecanum_wheel name="rear_right"  x="-0.08" y="-0.09"/>
+  <!-- Mecanum Wheel Orientation (X configuration) -->
+  <!-- FL: / (1, -1, 0)  FR: \ (1, 1, 0) -->
+  <!-- RL: \ (1, 1, 0)   RR: / (1, -1, 0) -->
+  <xacro:mecanum_wheel name="front_left"  x="0.08"  y="0.09"  fdir="0.707 -0.707 0"/>
+  <xacro:mecanum_wheel name="front_right" x="0.08"  y="-0.09" fdir="0.707 0.707 0"/>
+  <xacro:mecanum_wheel name="rear_left"   x="-0.08" y="0.09"  fdir="0.707 0.707 0"/>
+  <xacro:mecanum_wheel name="rear_right"  x="-0.08" y="-0.09" fdir="0.707 -0.707 0"/>
 </robot>
